File: Mixed_Signal_Design/Power.kicad_sch (KiCad schematic)
At the start: 19 parts, among them J1 Barrel_Jack, U1 LM1117DT-5.0, U2 LM1117DT-5.0

Commit message: commit
Parts:
- D1, D3: footprint (none) -> SparkFun-LED:LED_0603_1608Metric
- FB1: footprint Ferrite_THT:LairdTech_28C0236-0JW-10 -> FB_MI0805K400R-10:FB_MI0805K400R-10
- R1, R2: footprint (none) -> Resistor_SMD:R_0402_1005Metric_Pad0.72x0.64mm_HandSolder
Changed lines of the file:
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@@
   (junction (at 168.148 107.188) (diameter 0) (color 0 0 0 0)
   )
+  (junction (at 75.946 125.984) (diameter 0) (color 0 0 0 0)
+  )
   (junction (at 173.99 47.498) (diameter 0) (color 0 0 0 0)
   )
@@
   (junction (at 163.068 121.158) (diameter 0) (color 0 0 0 0)
   )
+  (junction (at 182.626 119.888) (diameter 0) (color 0 0 0 0)
+  )
   (junction (at 205.486 107.188) (diameter 0) (color 0 0 0 0)
   )
@@
   (junction (at 75.946 122.174) (diameter 0) (color 0 0 0 0)
   )
+  (wire (pts (xy 75.946 125.984) (xy 75.946 128.27))
+    (stroke (width 0) (type default))
+  )
   (wire (pts (xy 168.91 47.498) (xy 173.99 47.498))
     (stroke (width 0) (type default))
@@
     (stroke (width 0) (type default))
   )
+  (wire (pts (xy 163.068 121.158) (xy 163.068 123.698))
+    (stroke (width 0) (type default))
+  )
   (wire (pts (xy 194.818 107.188) (xy 194.818 111.76))
     (stroke (width 0) (type default))
@@
     (stroke (width 0) (type default))
   )
-  (wire (pts (xy 163.068 121.158) (xy 163.068 123.698))
-    (stroke (width 0) (type default))
-  )
   (wire (pts (xy 79.248 49.276) (xy 84.074 49.276))
     (stroke (width 0) (type default))
@@
     (stroke (width 0) (type default))
   )
-  (wire (pts (xy 182.626 114.808) (xy 182.626 121.158))
+  (wire (pts (xy 182.626 114.808) (xy 182.626 119.888))
     (stroke (width 0) (type default))
   )
@@
     (stroke (width 0) (type default))
   )
+  (wire (pts (xy 182.626 119.888) (xy 182.626 121.158))
+    (stroke (width 0) (type default))
+  )
   (wire (pts (xy 211.328 61.468) (xy 211.328 59.69))
     (stroke (width 0) (type default))
@@
     (stroke (width 0) (type default))
   )
-  (wire (pts (xy 75.946 122.174) (xy 75.946 128.27))
+  (wire (pts (xy 75.946 122.174) (xy 75.946 125.984))
     (stroke (width 0) (type default))
   )
@@
       (effects (font (size 1.27 1.27)) (justify right))
     )
-    (property "Footprint" "" (at 223.266 62.992 0)
+    (property "Footprint" "SparkFun-LED:LED_0603_1608Metric" (at 223.266 62.992 0)
       (effects (font (size 1.27 1.27)) hide)
     )
@@
         (path "/41b0ee65-569f-42b7-9c7e-4c72efc7a072/bc3efce2-5871-40f7-ae58-b147de6ab15e"
           (reference "#PWR03") (unit 1)
+        )
+      )
+    )
+  )
+  (symbol (lib_id "power:PWR_FLAG") (at 182.626 119.888 90) (unit 1)
+    (in_bom yes) (on_board yes) (dnp no) (fields_autoplaced)
+    (property "Reference" "#FLG04" (at 180.721 119.888 0)
+      (effects (font (size 1.27 1.27)) hide)
+    )
+    (property "Value" "PWR_FLAG" (at 179.07 119.888 90)
+      (effects (font (size 1.27 1.27)) (justify left))
+    )
+    (property "Footprint" "" (at 182.626 119.888 0)
+      (effects (font (size 1.27 1.27)) hide)
+    )
+    (property "Datasheet" "~" (at 182.626 119.888 0)
+      (effects (font (size 1.27 1.27)) hide)
+    )
+    (pin "1")
+    (instances
+      (project "Mixed_Signal_Design"
+        (path "/41b0ee65-569f-42b7-9c7e-4c72efc7a072/bc3efce2-5871-40f7-ae58-b147de6ab15e"
+          (reference "#FLG04") (unit 1)
         )
       )
@@
     (in_bom yes) (on_board yes) (dnp no) (fields_autoplaced)
     (property "Reference" "R2" (at 219.71 112.268 0)
-      (effects (font (size 1.27 1.27)) (justify left))
+      (effects (font (size 1.27 1.27) italic) (justify left))
     )
     (property "Value" "3.3K" (at 219.71 114.808 0)
       (effects (font (size 1.27 1.27)) (justify left))
     )
-    (property "Footprint" "" (at 215.646 113.538 90)
+    (property "Footprint" "Resistor_SMD:R_0402_1005Metric_Pad0.72x0.64mm_HandSolder" (at 215.646 113.538 90)
       (effects (font (size 1.27 1.27)) hide)
     )
@@
     )
   )
+  (symbol (lib_id "power:PWR_FLAG") (at 75.946 125.984 90) (unit 1)
+    (in_bom yes) (on_board yes) (dnp no) (fields_autoplaced)
+    (property "Reference" "#FLG03" (at 74.041 125.984 0)
+      (effects (font (size 1.27 1.27)) hide)
+    )
+    (property "Value" "PWR_FLAG" (at 72.39 125.984 90)
+      (effects (font (size 1.27 1.27)) (justify left))
+    )
+    (property "Footprint" "" (at 75.946 125.984 0)
+      (effects (font (size 1.27 1.27)) hide)
+    )
+    (property "Datasheet" "~" (at 75.946 125.984 0)
+      (effects (font (size 1.27 1.27)) hide)
+    )
+    (pin "1")
+    (instances
+      (project "Mixed_Signal_Design"
+        (path "/41b0ee65-569f-42b7-9c7e-4c72efc7a072/bc3efce2-5871-40f7-ae58-b147de6ab15e"
+          (reference "#FLG03") (unit 1)
+        )
+      )
+    )
+  )
   (symbol (lib_id "Regulator_Linear:LM1117DT-5.0") (at 182.626 107.188 0) (unit 1)
     (in_bom yes) (on_board yes) (dnp no) (fields_autoplaced)
@@
       (effects (font (size 1.27 1.27)))
     )
-    (property "Footprint" "Ferrite_THT:LairdTech_28C0236-0JW-10" (at 67.056 110.49 90)
+    (property "Footprint" "FB_MI0805K400R-10:FB_MI0805K400R-10" (at 67.056 110.49 90)
       (effects (font (size 1.27 1.27)) hide)
     )
@@
       (effects (font (size 1.27 1.27)) (justify right))
     )
-    (property "Footprint" "" (at 217.424 122.682 0)
+    (property "Footprint" "SparkFun-LED:LED_0603_1608Metric" (at 217.424 122.682 0)
       (effects (font (size 1.27 1.27)) hide)
     )
@@
       (effects (font (size 1.27 1.27)) (justify left))
     )
-    (property "Footprint" "" (at 221.488 53.848 90)
-      (effects (font (size 1.27 1.27)) hide)
-    )
+    (property "Footprint" "Resistor_SMD:R_0402_1005Metric_Pad0.72x0.64mm_HandSolder" (at 221.488 53.848 90)
+      (effects (font (size 1.27 1.27)) hide)
+    )
