File: Mixed_Signal_Design/_autosave-Mixed_Signal_Design.kicad_pcb (KiCad board)
At the start: 4 copper layers, 53.5 x 39.8 mm, 43 parts, among them J1 Barrel_Jack, J2 AVR-ISP-6, J4 Conn_01x08_Pin, SW1 RESET, U1 LM1117DT-5.0, U2 LM1117DT-5.0, U4 ATmega8L-8A, Y1 16MHz

Commit message: commit
Routing:
- net GNDD: vias 34 -> 46
