File: Mixed_Signal_Design/connectors.kicad_sch (KiCad schematic)
At the start: 0 parts

Commit message: commit
Parts:
- added FID1, FID2, FID3: Fiducial, Fiducial:Fiducial_0.75mm_Mask1.5mm, symbol Mechanical:Fiducial
- added H1, H2, H3, H4: MountingHole_Pad, MountingHole:MountingHole_2.2mm_M2_ISO7380_Pad, symbol Mechanical:MountingHole_Pad
- added J2: AVR-ISP-6, Connector_PinHeader_2.54mm:PinHeader_1x06_P2.54mm_Vertical, symbol Connector:AVR-ISP-6
- added J4: Conn_01x08_Pin, Connector_PinSocket_2.54mm:PinSocket_1x08_P2.54mm_Vertical, symbol Connector:Conn_01x08_Pin
Connections:
- new net +3V3D: J2.2 (VCC)
- new net ADC1: J4.1 (Pin_1)
- new net ADC2: J4.2 (Pin_2)
- new net GNDD: H1.1, H2.1, H3.1, H4.1, J2.6 (GND)
- new net PB3: J2.4 (MOSI)
- new net PB4: J2.1 (MISO)
- new net PB5: J2.3 (SCK)
- new net PC0: J4.3 (Pin_3)
- new net PC1: J4.4 (Pin_4)
- new net PC2: J4.5 (Pin_5)
- new net PC3: J4.6 (Pin_6)
- new net PC4: J4.7 (Pin_7)
- new net PC5: J4.8 (Pin_8)
- new net RST: J2.5 (~{RST})
